Commit message: more realistic vehicle params, better rendering

File: src/simulation/assets/vehicles/tractor_trailer.urdf (robot description, URDF)
Before this commit: robot tractor_trailer, 10 links, 9 joints
Links:
- link base_link: geometry collision box size=3.85 1.4 0.32; visual box size=3.85 1.4 0.32
- link front_left_wheel_link: geometry collision cylinder length=0.14 radius=0.33; visual cylinder length=0.14 radius=0.33
- link front_right_wheel_link: geometry collision cylinder length=0.14 radius=0.33; visual cylinder length=0.14 radius=0.33
- link rear_left_wheel_link: geometry collision cylinder length=0.14 radius=0.33; visual cylinder length=0.14 radius=0.33
- link rear_right_wheel_link: geometry collision cylinder length=0.14 radius=0.33; visual cylinder length=0.14 radius=0.33
- link trailer_left_wheel_link: geometry collision cylinder length=0.14 radius=0.33; visual cylinder length=0.14 radius=0.33
- link trailer_link: geometry collision box size=3.4 1.4 0.28; visual box size=3.4 1.4 0.3
- link trailer_right_wheel_link: geometry collision cylinder length=0.14 radius=0.33; visual cylinder length=0.14 radius=0.33
Joints:
- joint front_left_steer: origin xyz=0.92 0.50 0.12 rpy=0 0 0 -> xyz=1.45 0.50 0.12 rpy=0 0 0
- joint front_right_steer: origin xyz=0.92 -0.50 0.12 rpy=0 0 0 -> xyz=1.45 -0.50 0.12 rpy=0 0 0
- joint hitch: limit lower=-1.5708 upper=1.5708 effort=0 velocity=10 -> lower=-2.0944 upper=2.0944 effort=0 velocity=10; origin xyz=-1.0 0 0 rpy=0 0 0 -> xyz=-2.3 0 0 rpy=0 0 0
- joint rear_left_wheel: origin xyz=-0.92 0.50 0.12 rpy=0 0 0 -> xyz=-1.60 0.50 0.12 rpy=0 0 0
- joint rear_right_wheel: origin xyz=-0.92 -0.50 0.12 rpy=0 0 0 -> xyz=-1.60 -0.50 0.12 rpy=0 0 0
- joint trailer_left_wheel: origin xyz=-3.0 0.50 0.12 rpy=0 0 0 -> xyz=-2.5 0.50 0.12 rpy=0 0 0
- joint trailer_right_wheel: origin xyz=-3.0 -0.50 0.12 rpy=0 0 0 -> xyz=-2.5 -0.50 0.12 rpy=0 0 0
