Commit message: benchmarking implemented, mppi satisfactory, smppi bad

File: src/simulation/assets/vehicles/simple_racecar.urdf (robot description, URDF)
Before this commit: robot simple_racecar, 7 links, 6 joints
Links:
- link front_left_wheel_link: geometry collision cylinder length=0.14 radius=0.33; visual cylinder length=0.14 radius=0.33
- link front_right_wheel_link: geometry collision cylinder length=0.14 radius=0.33; visual cylinder length=0.14 radius=0.33
- link rear_left_wheel_link: geometry collision cylinder length=0.14 radius=0.33; visual cylinder length=0.14 radius=0.33
- link rear_right_wheel_link: geometry collision cylinder length=0.14 radius=0.33; visual cylinder length=0.14 radius=0.33

Commit message: fix smppi diff bug, tuning

File: src/simulation/assets/vehicles/simple_racecar.urdf (robot description, URDF)
Before this commit: robot simple_racecar, 7 links, 6 joints
Links:
- link base_link: geometry collision box size=2.4 1.1 0.28; visual box size=2.4 1.2 0.28
